File: schematics/USBHub/USBHub.sch (KiCad schematic (older format))
At the start: 35 parts, among them J1 USB_A_STACKED, J2 USB_A_STACKED, J3 USB_B, J6 Screw_Terminal_01x02, U1 FE1.1, U2 AP2411, Y1 12Mhz

Commit message: Fixed up USBHub symbol and footprint library
Parts:
- J1, J2: symbol MiSTer-Custom:USB_A_STACKED -> USBHub:USB_A_STACKED
- U1: footprint MiSTer-G3:FE1_1_QFP48 -> USBHub:FE1_1_QFP48; symbol MiSTer-Custom:FE1.1 -> USBHub:FE1.1
- U2: footprint MiSTer-G3:AP24x1_SO8_HandSolder -> USBHub:AP24x1_SO8_HandSolder; symbol MiSTer-Custom:AP2411 -> USBHub:AP2411
Changed lines of the file:
@@
 $EndDescr
 $Comp
-L MiSTer-Custom:FE1.1 U1
+L USBHub:FE1.1 U1
 U 1 1 61248B22
 P 2800 4100
 F 0 "U1" H 2800 2611 50  0000 C CNN
 F 1 "FE1.1" H 2800 2520 50  0000 C CNN
-F 2 "MiSTer-G3:FE1_1_QFP48" H 2800 4150 50  0001 C CNN
+F 2 "USBHub:FE1_1_QFP48" H 2800 4150 50  0001 C CNN
 F 3 "" H 2800 4150 50  0001 C CNN
 	1    2800 4100
@@
 	6300 3050 6400 3050
 $Comp
-L MiSTer-Custom:AP2411 U2
+L USBHub:AP2411 U2
 U 1 1 6134CC47
 P 7550 3200
 F 0 "U2" H 7550 3715 50  0000 C CNN
 F 1 "AP2411" H 7550 3624 50  0000 C CNN
-F 2 "MiSTer-G3:AP24x1_SO8_HandSolder" H 7500 3300 50  0001 C CNN
+F 2 "USBHub:AP24x1_SO8_HandSolder" H 7500 3300 50  0001 C CNN
 F 3 "" H 7500 3300 50  0001 C CNN
 	1    7550 3200
@@
 Connection ~ 8850 2950
 $Comp
-L MiSTer-Custom:USB_A_STACKED J1
+L USBHub:USB_A_STACKED J1
 U 1 1 613D0FEB
 P 1350 1250
@@
 Connection ~ 1350 2000
 $Comp
-L MiSTer-Custom:USB_A_STACKED J1
+L USBHub:USB_A_STACKED J1
 U 2 1 613DE136
 P 2400 1250
@@
 Connection ~ 2400 2000
 $Comp
-L MiSTer-Custom:USB_A_STACKED J2
+L USBHub:USB_A_STACKED J2
 U 1 1 613EA626
 P 4300 1250
@@
 Connection ~ 3350 2000
 $Comp
-L MiSTer-Custom:USB_A_STACKED J2
+L USBHub:USB_A_STACKED J2
 U 2 1 613EC447
 P 3350 1250

Commit message: Schematic changes
Reworked Rocky Hills j22 adaptor, removed microphone, added JST headers for speakers, buttons and headphones.
Updated USBHub for FE1.1 5V doesn't go through the current limiting switch
Connections:
- net VBUS: no longer C10.1, U1.38 (VD5_IN)
- net VD5: now reaches C7.1, J6.2 (Pin_2), U2.2 (IN), U2.3 (IN)
- net VD5: now also C10.1, U1.38 (VD5_IN)
Changed lines of the file:
@@
 Connection ~ 6350 2950
 Wire Wire Line
-	6350 2950 6600 2950
-Text GLabel 9000 3150 2    50   Output ~ 0
+	6350 2950 6500 2950
+Text GLabel 6700 2850 2    50   Output ~ 0
 VD5
 Wire Wire Line
 	4000 3300 4800 3300
-Wire Wire Line
-	8850 2950 8850 3150
-Wire Wire Line
-	8850 3150 9000 3150
-Wire Wire Line
-	8550 2950 8850 2950
-Wire Wire Line
-	8850 2950 9000 2950
-Connection ~ 8850 2950
 $Comp
 L USBHub:USB_A_STACKED J1
@@
 Text Label 3250 6200 0    50   ~ 0
 DU-
+Wire Wire Line
+	6500 2950 6500 2850
+Wire Wire Line
+	6500 2850 6700 2850
+Connection ~ 6500 2950
+Wire Wire Line
+	6500 2950 6600 2950
+Wire Wire Line
+	8550 2950 9000 2950
 $EndSCHEMATC
