File: schematics/USBHub/USBHub.kicad_sch (KiCad schematic)
At the start: 35 parts

Commit message: Update part numbers
Parts:
- C1, C2, C3, C4, C5, C6, C9: value (none) -> 10u; footprint (none) -> Capacitor_SMD:C_0603_1608Metric_Pad1.08x0.95mm_HandSolder; Part# (none) -> 1276-1038-1-ND; Vendor (none) -> digikey
- C10, C11, C12, C13, C14, C15, C16, C17, C18, C7, C8: value (none) -> 100n; footprint (none) -> Capacitor_SMD:C_0603_1608Metric_Pad1.08x0.95mm_HandSolder; Part# (none) -> 1276-1935-1-ND; Vendor (none) -> digikey
- H1, H2, H3, H4: value (none) -> MountingHole_Pad; footprint (none) -> MountingHole:MountingHole_3.2mm_M3_Pad_Via
- J1, J2: value (none) -> USB_A_STACKED; footprint (none) -> Connector_USB:USB_A_Wuerth_61400826021_Horizontal_Stacked; Part# (none) -> 2057-USB-A-D-RA-ND; Vendor (none) -> digikey
- J3: value (none) -> USB_B; footprint (none) -> Connector_USB:USB_B_OST_USB-B1HSxx_Horizontal; Part# (none) -> ED2983-ND; Vendor (none) -> digikey
- J6: value (none) -> Screw_Terminal_01x02; footprint (none) -> TerminalBlock_Phoenix:TerminalBlock_Phoenix_MPT-0,5-2-2.54_1x02_P2.54mm_Horizontal; Part# (none) -> 277-1273-ND; Vendor (none) -> digikey
- R1: value (none) -> 2.7K; footprint (none) -> Resistor_SMD:R_0603_1608Metric_Pad0.98x0.95mm_HandSolder; Part# (none) -> 311-2.7KGRCT-ND; Vendor (none) -> digikey
- R2, R3, R5: value (none) -> 100k; footprint (none) -> Resistor_SMD:R_0603_1608Metric_Pad0.98x0.95mm_HandSolder; Part# (none) -> 311-100KGRCT-ND; Vendor (none) -> digikey
- R4: value (none) -> 47k; footprint (none) -> Resistor_SMD:R_0603_1608Metric_Pad0.98x0.95mm_HandSolder; Part# (none) -> 311-47KGRCT-ND; Vendor (none) -> digikey
- R6: value (none) -> 10k; footprint (none) -> Resistor_SMD:R_0603_1608Metric_Pad0.98x0.95mm_HandSolder; Part# (none) -> 311-10KGRCT-ND; Vendor (none) -> digikey
- U1: value (none) -> FE1.1; footprint (none) -> USBHub:FE1_1_QFP48
- U2: value (none) -> AP2411; footprint (none) -> USBHub:AP24x1_SO8_HandSolder; Part# (none) -> AP2411S-13DICT-ND; Vendor (none) -> digikey
- Y1: value (none) -> 12Mhz; footprint (none) -> Crystal:Crystal_SMD_0603-2Pin_6.0x3.5mm_HandSoldering; Part# (none) -> F61200046CT-ND; Vendor (none) -> digikey
