File: schematics/MiSTer-G3/MiSTer-G3.sch (KiCad schematic (older format))
At the start: 37 parts, among them J1 Apple J20, J2 VGA Input, J3 Audio, J4 I2S, J5 Power, J6 Rotary Encoder, U1 TPA6021A4N, U2 UDA1334A, U3 LCC110

Commit message: Headers and routing
Added JST header for mister buttons
Split screw terminals into separate JST headers for speakers, headphones and front panel.
Added rotary encoder button

Re-routed pcb
Parts:
- removed J3: Audio, TerminalBlock_Phoenix:TerminalBlock_Phoenix_MPT-0,5-8-2.54_1x08_P2.54mm_Horizontal, symbol Connector:Screw_Terminal_01x08
- removed J5: Power, TerminalBlock_Phoenix:TerminalBlock_Phoenix_MPT-0,5-8-2.54_1x08_P2.54mm_Horizontal, symbol Connector:Screw_Terminal_01x08
- added J3: Speaker, Connector_JST:JST_XH_B4B-XH-A_1x04_P2.50mm_Vertical, symbol Connector:Conn_01x04_Male
- added J5: Power, Connector_JST:JST_XH_B4B-XH-A_1x04_P2.50mm_Vertical, symbol Connector:Conn_01x04_Male
- added J7: Headphones, Connector_JST:JST_XH_B4B-XH-A_1x04_P2.50mm_Vertical, symbol Connector:Conn_01x04_Male
- added J8: Front Panel, Connector_JST:JST_XH_B4B-XH-A_1x04_P2.50mm_Vertical, symbol Connector:Conn_01x04_Male
- added J9: Buttons, Connector_JST:JST_XH_B5B-XH-A_1x05_P2.50mm_Vertical, symbol Connector:Conn_01x05_Male
- J6: footprint Connector_JST:JST_XH_B3B-XH-A_1x03_P2.50mm_Vertical -> Connector_JST:JST_XH_B4B-XH-A_1x04_P2.50mm_Vertical; symbol Connector:Conn_01x03_Male -> Connector:Conn_01x04_Male
Connections:
- net +5V: now also J5.1 (Pin_1)
- net AMBER_LED: now also A1.6 (D3), J8.2 (Pin_2); no longer A1.8 (D5)
- net AMP_ACTIVE: now also A1.15 (MISO); no longer A1.10 (D7)
- net DCO: now also J5.3 (Pin_3)
- net GND: now also J5.2 (Pin_2), J7.4 (Pin_4), J8.4 (Pin_4), J9.5 (Pin_5)
- net GREEN_LED: now also A1.5 (D2), J8.1 (Pin_1); no longer A1.7 (D4)
- net LHEAD: now also J7.2 (Pin_2)
- net LSPKR+: now also J3.3 (Pin_3)
- net LSPKR-: now also J3.4 (Pin_4)
- net POWER_BTN: now also A1.7 (D4), J8.3 (Pin_3); no longer A1.9 (D6)
- net PROT: now also J5.4 (Pin_4)
- net RHEAD: now also J7.1 (Pin_1)
- net ROT_A: now also A1.26 (A7); no longer A1.5 (D2)
- net ROT_B: now also A1.25 (A6); no longer A1.6 (D3)
- net RSPKR+: now also J3.1 (Pin_1)
- net RSPKR-: now also J3.2 (Pin_2)
- net SHEAD: now also J7.3 (Pin_3)
- net ROT_BTN: now reaches A1.11 (D8)
- net ROT_BTN: now also J6.4 (Pin_4)
- net at A1.12 (D9): no longer R6.1
- net at A1.13 (D10): now also R6.1
- new net BTN_OSD: A1.9 (D6), J9.2 (Pin_2)
- new net BTN_RESET: A1.8 (D5), J9.3 (Pin_3)
- new net BTN_USER: A1.10 (D7), J9.1 (Pin_1)
- no-connect marks 33 -> 30
Other:
- moved on the sheet: C10, J4, R6

Commit message: Headphone sense
Added second sense wire from j22 board since they can't be combined.
Send sense inputs to arduino and control SE/~BTL signal from there. This will allow different volume settings for each mode.
Re-route.
Fix silkscreen labels
Parts:
- added R10, R11: 100k, Resistor_THT:R_Axial_DIN0207_L6.3mm_D2.5mm_P10.16mm_Horizontal, symbol Device:R
- J7: footprint Connector_JST:JST_XH_B4B-XH-A_1x04_P2.50mm_Vertical -> Connector_JST:JST_XH_B5B-XH-A_1x05_P2.50mm_Vertical; symbol Connector:Conn_01x04_Male -> Connector:Conn_01x05_Male
Connections:
- net +5V: no longer R2.1
- net 5V_MCU: now also R2.1, R11.1
- net GND: now also J7.5 (Pin_5); no longer J7.4 (Pin_4)
- net AMP_SE: now reaches U1.19 (SE/~BTL)
- net AMP_SE: now also A1.14 (MOSI); no longer R1.2
- net ~HEAD_DETECT1: now reaches A1.20 (A1)
- net ~HEAD_DETECT1: now also R1.2
- net ~HEAD_DETECT2: now reaches A1.21 (A2)
- net ~HEAD_DETECT2: now also R10.2
- net SHEAD renamed SHEAD1
- new net SHEAD2: J7.4 (Pin_4), R10.1, R11.2
- no-connect marks 30 -> 27
Other:
- moved on the sheet: R1, R2
Changed lines of the file:
@@
 Connection ~ 5650 6150
-$Comp
-L power:+5V #PWR017
-U 1 1 60D318B3
-P 4950 4800
-F 0 "#PWR017" H 4950 4650 50  0001 C CNN
-F 1 "+5V" H 4965 4973 50  0000 C CNN
-F 2 "" H 4950 4800 50  0001 C CNN
-F 3 "" H 4950 4800 50  0001 C CNN
-	1    4950 4800
-	1    0    0    -1
-$EndComp
-$Comp
-L Device:R R2
-U 1 1 60D322F3
-P 4950 4950
-F 0 "R2" H 5020 4996 50  0000 L CNN
-F 1 "100k" H 5020 4905 50  0000 L CNN
-F 2 "Resistor_THT:R_Axial_DIN0207_L6.3mm_D2.5mm_P10.16mm_Horizontal" V 4880 4950 50  0001 C CNN
-F 3 "~" H 4950 4950 50  0001 C CNN
-	1    4950 4950
-	1    0    0    -1
-$EndComp
-$Comp
-L Device:R R1
-U 1 1 60D3263B
-P 4550 4950
-F 0 "R1" V 4343 4950 50  0000 C CNN
-F 1 "100k" V 4434 4950 50  0000 C CNN
-F 2 "Resistor_THT:R_Axial_DIN0207_L6.3mm_D2.5mm_P10.16mm_Horizontal" V 4480 4950 50  0001 C CNN
-F 3 "~" H 4550 4950 50  0001 C CNN
-	1    4550 4950
-	0    1    1    0
-$EndComp
-Text GLabel 5150 5100 2    50   Input ~ 0
-SHEAD
-Wire Wire Line
-	4700 4950 4800 4950
-Wire Wire Line
-	4800 4950 4800 5100
-Wire Wire Line
-	4800 5100 4950 5100
-Wire Wire Line
-	4950 5100 5150 5100
-Connection ~ 4950 5100
 $Comp
 L Device:CP1 C1
@@
 Text GLabel 5900 5700 2    50   Input ~ 0
 AMP_ACTIVE
-Wire Wire Line
-	4400 5100 4650 5100
 Wire Wire Line
 	4400 5250 4600 5250
@@
 LHEAD
 Text GLabel 3400 950  2    50   Output ~ 0
-SHEAD
+SHEAD1
 $Comp
 L power:GND #PWR013
 U 1 1 60D3FF2A
-P 3550 1100
-F 0 "#PWR013" H 3550 850 50  0001 C CNN
-F 1 "GND" H 3555 927 50  0000 C CNN
-F 2 "" H 3550 1100 50  0001 C CNN
-F 3 "" H 3550 1100 50  0001 C CNN
-	1    3550 1100
+P 3550 1200
+F 0 "#PWR013" H 3550 950 50  0001 C CNN
+F 1 "GND" H 3555 1027 50  0000 C CNN
+F 2 "" H 3550 1200 50  0001 C CNN
+F 3 "" H 3550 1200 50  0001 C CNN
+	1    3550 1200
 	1    0    0    -1
 $EndComp
@@
 	1    0    0    -1
 $EndComp
-Wire Wire Line
-	4650 5100 4650 5250
 Wire Wire Line
 	4650 5250 4750 5250
@@
 NoConn ~ 8850 4000
 NoConn ~ 8850 4100
-NoConn ~ 8850 5300
 NoConn ~ 8850 5500
 NoConn ~ 9850 5100
-NoConn ~ 9850 5000
 NoConn ~ 9850 4600
 NoConn ~ 9850 4300
@@
 	1    0    0    -1
 $EndComp
-NoConn ~ 9850 4900
 $Comp
 L Device:R_Small R9
@@
 $EndComp
 $Comp
-L Connector:Conn_01x04_Male J7
+L Connector:Conn_01x05_Male J7
 U 1 1 60F03800
-P 3200 850
-F 0 "J7" H 3308 1131 50  0000 C CNN
-F 1 "Headphones" H 3308 1040 50  0000 C CNN
-F 2 "Connector_JST:JST_XH_B4B-XH-A_1x04_P2.50mm_Vertical" H 3200 850 50  0001 C CNN
-F 3 "~" H 3200 850 50  0001 C CNN
-	1    3200 850
-	1    0    0    -1
-$EndComp
-Wire Wire Line
-	3400 1050 3550 1050
-Wire Wire Line
-	3550 1050 3550 1100
+P 3200 950
+F 0 "J7" H 3300 1350 50  0000 C CNN
+F 1 "Headphones" H 3400 1250 50  0000 C CNN
+F 2 "Connector_JST:JST_XH_B5B-XH-A_1x05_P2.50mm_Vertical" H 3200 950 50  0001 C CNN
+F 3 "~" H 3200 950 50  0001 C CNN
+	1    3200 950
+	1    0    0    -1
+$EndComp
+Wire Wire Line
+	3550 1150 3550 1200
 $Comp
 L Connector:Conn_01x05_Male J9
@@
 NoConn ~ 8850 5000
 NoConn ~ 12100 6550
+Wire Wire Line
+	4650 5100 4650 5250
+Wire Wire Line
+	4400 5100 4650 5100
+Wire Wire Line
+	4100 3050 4300 3050
+Text GLabel 4300 3050 2    50   Input ~ 0
+SHEAD1
+$Comp
+L Device:R R1
+U 1 1 60D3263B
+P 3850 3050
+F 0 "R1" V 3643 3050 50  0000 C CNN
+F 1 "100k" V 3734 3050 50  0000 C CNN
+F 2 "Resistor_THT:R_Axial_DIN0207_L6.3mm_D2.5mm_P10.16mm_Horizontal" V 3780 3050 50  0001 C CNN
+F 3 "~" H 3850 3050 50  0001 C CNN
+	1    3850 3050
+	0    1    1    0
+$EndComp
+$Comp
+L Device:R R2
+U 1 1 60D322F3
+P 4100 2900
+F 0 "R2" H 4170 2946 50  0000 L CNN
+F 1 "100k" H 4170 2855 50  0000 L CNN
+F 2 "Resistor_THT:R_Axial_DIN0207_L6.3mm_D2.5mm_P10.16mm_Horizontal" V 4030 2900 50  0001 C CNN
+F 3 "~" H 4100 2900 50  0001 C CNN
+	1    4100 2900
+	1    0    0    -1
+$EndComp
+Wire Wire Line
+	4000 3050 4100 3050
+Connection ~ 4100 3050
+Wire Wire Line
+	4100 3250 4300 3250
+Text GLabel 4300 3250 2    50   Input ~ 0
+SHEAD2
+$Comp
+L Device:R R10
+U 1 1 61007E6C
+P 3850 3250
+F 0 "R10" V 3643 3250 50  0000 C CNN
+F 1 "100k" V 3734 3250 50  0000 C CNN
+F 2 "Resistor_THT:R_Axial_DIN0207_L6.3mm_D2.5mm_P10.16mm_Horizontal" V 3780 3250 50  0001 C CNN
+F 3 "~" H 3850 3250 50  0001 C CNN
+	1    3850 3250
+	0    1    -1   0
+$EndComp
+$Comp
+L Device:R R11
+U 1 1 61007E76
+P 4100 3400
+F 0 "R11" H 4170 3446 50  0000 L CNN
+F 1 "100k" H 4170 3355 50  0000 L CNN
+F 2 "Resistor_THT:R_Axial_DIN0207_L6.3mm_D2.5mm_P10.16mm_Horizontal" V 4030 3400 50  0001 C CNN
+F 3 "~" H 4100 3400 50  0001 C CNN
+	1    4100 3400
+	1    0    0    1
+$EndComp
+Wire Wire Line
+	4000 3250 4100 3250
+Connection ~ 4100 3250
+Text GLabel 4550 4950 2    50   Input ~ 0
+AMP_SE
+Wire Wire Line
+	4400 4950 4550 4950
+Wire Wire Line
+	3400 1150 3550 1150
+Text GLabel 3400 1050 2    50   Output ~ 0
+SHEAD2
+Text GLabel 8500 5600 0    50   Output ~ 0
+AMP_SE
+Wire Wire Line
+	8850 5300 8650 5300
+Wire Wire Line
+	8650 5300 8650 5600
+Wire Wire Line
+	8650 5600 8500 5600
+Text GLabel 3600 3050 0    50   Input ~ 0
+~HEAD_DETECT1
+Text GLabel 3600 3250 0    50   Input ~ 0
+~HEAD_DETECT2
+Wire Wire Line
+	3600 3050 3700 3050
+Wire Wire Line
+	3600 3250 3700 3250
+Text GLabel 10000 4950 2    50   Output ~ 0
+~HEAD_DETECT1
+Text GLabel 10000 5100 2    50   Output ~ 0
+~HEAD_DETECT2
+Wire Wire Line
+	9850 4900 9950 4900
+Wire Wire Line
+	9950 4900 9950 4950
+Wire Wire Line
+	9950 4950 10000 4950
+Wire Wire Line
+	9850 5000 9950 5000
+Wire Wire Line
+	9950 5000 9950 5100
+Wire Wire Line
+	9950 5100 10000 5100
+Text GLabel 4100 3550 3    50   Output ~ 0
+5V_MCU
+Text GLabel 4100 2750 1    50   Output ~ 0
+5V_MCU
 $EndSCHEMATC

Commit message: Code and schematic changes
Fixed incorrect routing for decoupling caps
Updated code to handle headphones, power button and mister buttons.
Parts:
- A1: Part# (none) -> S7013-ND; Vendor (none) -> digikey
- C1, C11, C12, C2, C4, C5, C6, C7: Part# (none) -> 478-8779-1-ND; Vendor (none) -> digikey
- C10: Part# (none) -> 445-173588-1-ND; Vendor (none) -> digikey
- C3: Part# (none) -> 493-15134-ND; Vendor (none) -> digikey
- C8, C9: Part# (none) -> 493-3180-ND; Vendor (none) -> digikey
- D1, D2: Part# (none) -> 1N5819-E3/54GICT-ND; Vendor (none) -> digikey
- J1: Part# (none) -> SAM1068-10-ND; Vendor (none) -> digikey
- J2: Part# (none) -> L77HDE15SD1CH4F-ND; Vendor (none) -> digikey
- J3, J5, J6, J8: Part# (none) -> 455-2249-ND; Vendor (none) -> digikey
- J4, J7, J9: Part# (none) -> 455-2270-ND; Vendor (none) -> digikey
- R1, R10, R11, R2: Part# (none) -> 100KQBK-ND; Vendor (none) -> digikey
- R3, R6: Part# (none) -> 10KQBK-ND; Vendor (none) -> digikey
- R4, R5: Part# (none) -> 1.0KQBK-ND; Vendor (none) -> digikey
- R7, R8: Part# (none) -> 4.7KQBK-ND; Vendor (none) -> digikey
- R9: Part# (none) -> 220QBK-ND; Vendor (none) -> digikey
- U1: Part# (none) -> 296-18249-5-ND; Vendor (none) -> digikey
- U2: Part# (none) -> 3678; Vendor (none) -> adafruit
- U3: Part# (none) -> CLA106-ND; Vendor (none) -> digikey
