File: schematics/imac_g3_slot_loading_J22_adapter_board/imac_g3_slot_loading_J22_adapter_board.sch (KiCad schematic (older format))
At the start: 8 parts, among them J1 Conn_02x13_Odd_Even, J2 AC Power, J3 Conn_01x04_Male, J4 Conn_01x04_Male, J5 Conn_01x04_Male

Commit message: Headphone sense
Added second sense wire from j22 board since they can't be combined.
Send sense inputs to arduino and control SE/~BTL signal from there. This will allow different volume settings for each mode.
Re-route.
Fix silkscreen labels
Parts:
- J5: footprint Connector_JST:JST_XH_B4B-XH-A_1x04_P2.50mm_Vertical -> Connector_JST:JST_XH_B5B-XH-A_1x05_P2.50mm_Vertical; symbol Connector:Conn_01x04_Male -> Connector:Conn_01x05_Male
Connections:
- net GNDREF: now also J5.5 (Pin_5); no longer J5.4 (Pin_4)
- net HEADPHONE_1_SENSE: no longer J1.7 (Pin_7)
- new net HEADPHONE_2_SENSE: J1.7 (Pin_7), J5.4 (Pin_4)
Changed lines of the file:
@@
 	1200 2100 1550 2100
 $Comp
-L Connector:Conn_01x04_Male J5
+L Connector:Conn_01x05_Male J5
 U 1 1 60F48977
-P 900 2750
-F 0 "J5" H 1008 3031 50  0000 C CNN
-F 1 "Conn_01x04_Male" H 1008 2940 50  0000 C CNN
-F 2 "Connector_JST:JST_XH_B4B-XH-A_1x04_P2.50mm_Vertical" H 900 2750 50  0001 C CNN
-F 3 "~" H 900 2750 50  0001 C CNN
-	1    900  2750
+P 900 2850
+F 0 "J5" H 1008 3131 50  0000 C CNN
+F 1 "Conn_01x04_Male" H 1000 3250 50  0000 C CNN
+F 2 "Connector_JST:JST_XH_B5B-XH-A_1x05_P2.50mm_Vertical" H 900 2850 50  0001 C CNN
+F 3 "~" H 900 2850 50  0001 C CNN
+	1    900  2850
 	1    0    0    -1
 $EndComp
@@
 HEADPHONE_LEFT
 Text Label 1400 2850 0    50   ~ 0
-HEADPHONE_SENSE
-Text Label 1400 2950 0    50   ~ 0
+HEADPHONE_1_SENSE
+Text Label 1400 3050 0    50   ~ 0
 HEADPHONE_1_&_2_GND
 Wire Wire Line
@@
 Text Label 3350 3250 2    50   ~ 0
 HEADPHONE_LEFT
-Text Label 3350 3600 2    50   ~ 0
-HEADPHONE_SENSE
 Text Label 3550 2900 0    50   ~ 0
 HEADPHONE_2_RIGHT
@@
 Text Label 3550 3350 0    50   ~ 0
 HEADPHONE_2_LEFT
-Text Label 3550 3600 0    50   ~ 0
-HEADPHONE_1_SENSE
-Text Label 3550 3700 0    50   ~ 0
-HEADPHONE_2_SENSE
 Wire Wire Line
 	3350 2900 3500 2900
@@
 Wire Wire Line
 	3500 2900 3550 2900
-Wire Wire Line
-	3350 3600 3500 3600
-Wire Wire Line
-	3500 3600 3500 3700
-Wire Wire Line
-	3500 3700 3550 3700
-Connection ~ 3500 3600
-Wire Wire Line
-	3500 3600 3550 3600
 Wire Wire Line
 	3350 3250 3500 3250
@@
 Text Label 8800 4350 2    50   ~ 0
 HEADPHONE_1_&_2_GND
+Wire Wire Line
+	1100 3050 1400 3050
+Text Label 1400 2950 0    50   ~ 0
+HEADPHONE_2_SENSE
 $EndSCHEMATC

Commit message: Code and schematic changes
Fixed incorrect routing for decoupling caps
Updated code to handle headphones, power button and mister buttons.
Parts:
- J2: Part# 277-9080-ND -> 277-6405-ND
- J3, J4: Part# (none) -> 455-2249-ND; Vendor (none) -> digikey
- J5: Part# (none) -> 455-2270-ND; Vendor (none) -> digikey
Changed lines of the file:
@@
 F 3 "https://www.phoenixcontact.com/pxc-oc-itemdetail-pdf-web/eshop?lineItemType=LineItem&UID=1935857" H 1000 2200 50  0001 C CNN
 F 4 "digikey" H 1000 2200 50  0001 C CNN "Vendor"
-F 5 "277-9080-ND" H 1000 2200 50  0001 C CNN "Part#"
+F 5 "277-6405-ND" H 1000 2200 50  0001 C CNN "Part#"
 	1    1000 2200
 	-1   0    0    1
@@
 F 2 "Connector_JST:JST_XH_B4B-XH-A_1x04_P2.50mm_Vertical" H 900 950 50  0001 C CNN
 F 3 "~" H 900 950 50  0001 C CNN
+F 4 "digikey" H 900 950 50  0001 C CNN "Vendor"
+F 5 "455-2249-ND" H 900 950 50  0001 C CNN "Part#"
 	1    900  950
 	1    0    0    -1
@@
 F 2 "Connector_JST:JST_XH_B4B-XH-A_1x04_P2.50mm_Vertical" H 900 1600 50  0001 C CNN
 F 3 "~" H 900 1600 50  0001 C CNN
+F 4 "digikey" H 900 1600 50  0001 C CNN "Vendor"
+F 5 "455-2249-ND" H 900 1600 50  0001 C CNN "Part#"
 	1    900  1600
 	1    0    0    -1
@@
 Wire Wire Line
 	1200 2100 1550 2100
-$Comp
-L Connector:Conn_01x05_Male J5
-U 1 1 60F48977
-P 900 2850
-F 0 "J5" H 1008 3131 50  0000 C CNN
-F 1 "Conn_01x04_Male" H 1000 3250 50  0000 C CNN
-F 2 "Connector_JST:JST_XH_B5B-XH-A_1x05_P2.50mm_Vertical" H 900 2850 50  0001 C CNN
-F 3 "~" H 900 2850 50  0001 C CNN
-	1    900  2850
-	1    0    0    -1
-$EndComp
 Text Label 1400 2650 0    50   ~ 0
 HEADPHONE_RIGHT
@@
 Text Label 1400 2950 0    50   ~ 0
 HEADPHONE_2_SENSE
+$Comp
+L Connector:Conn_01x05_Male J5
+U 1 1 60F48977
+P 900 2850
+F 0 "J5" H 1008 3131 50  0000 C CNN
+F 1 "Conn_01x04_Male" H 1000 3250 50  0000 C CNN
+F 2 "Connector_JST:JST_XH_B5B-XH-A_1x05_P2.50mm_Vertical" H 900 2850 50  0001 C CNN
+F 3 "~" H 900 2850 50  0001 C CNN
+F 4 "digikey" H 900 2850 50  0001 C CNN "Vendor"
+F 5 "455-2270-ND" H 900 2850 50  0001 C CNN "Part#"
+	1    900  2850
+	1    0    0    -1
+$EndComp
 $EndSCHEMATC
